Commit message: Initial commit from cv_robot

File: urdf/cv_robot.urdf.xacro (robot description, xacro)
@@ -8,11 +8,7 @@
   </joint>
   <material name="chassis">     <color rgba="0.25 0.28 0.32 1"/></material>
-  <material name="teal">        <color rgba="0.11 0.72 0.55 1"/></material>
-  <material name="orange_rim">  <color rgba="1.00 0.55 0.10 1"/></material>
   <material name="dark_rubber"> <color rgba="0.18 0.18 0.18 1"/></material>
   <material name="top_cap">     <color rgba="0.35 0.38 0.42 1"/></material>
-  <material name="sensor_blue"> <color rgba="0.10 0.45 0.80 1"/></material>
-  <material name="white">       <color rgba="1.00 1.00 1.00 1"/></material>
-  <!-- Main chassis -->
+  <!-- Main chassis (cylinder) -->
   <link name="base_link">
     <visual>
@@ -32,84 +28,4 @@
     </inertial>
   </link>
-  <!-- Teal accent ring -->
-  <link name="accent_ring">
-    <visual>
-      <geometry>
-        <cylinder radius="0.37" length="0.018"/>
-      </geometry>
-      <material name="teal"/>
-    </visual>
-    <collision>
-      <geometry><cylinder radius="0.001" length="0.001"/></geometry>
-    </collision>
-    <inertial>
-      <mass value="0.05"/>
-      <inertia ixx="0.00005" ixy="0" ixz="0" iyy="0.00005" iyz="0" izz="0.00009"/>
-    </inertial>
-  </link>
-  <joint name="accent_ring_joint" type="fixed">
-    <parent link="base_link"/>
-    <child link="accent_ring"/>
-    <origin xyz="0 0 0.01" rpy="0 0 0"/>
-  </joint>
-  <!-- Top plate cap -->
-  <link name="top_plate">
-    <visual>
-      <geometry>
-        <cylinder radius="0.34" length="0.012"/>
-      </geometry>
-      <material name="top_cap"/>
-    </visual>
-    <collision>
-      <geometry><cylinder radius="0.001" length="0.001"/></geometry>
-    </collision>
-    <inertial>
-      <mass value="0.2"/>
-      <inertia ixx="0.0003" ixy="0" ixz="0" iyy="0.0003" iyz="0" izz="0.0006"/>
-    </inertial>
-  </link>
-  <joint name="top_plate_joint" type="fixed">
-    <parent link="base_link"/>
-    <child link="top_plate"/>
-    <origin xyz="0 0 0.036" rpy="0 0 0"/>
-  </joint>
-  <!-- Sensor dome -->
-  <link name="sensor_dome">
-    <visual>
-      <geometry><cylinder radius="0.09" length="0.05"/></geometry>
-      <material name="sensor_blue"/>
-    </visual>
-    <collision>
-      <geometry><cylinder radius="0.09" length="0.05"/></geometry>
-    </collision>
-    <inertial>
-      <mass value="0.25"/>
-      <inertia ixx="0.0008" ixy="0" ixz="0" iyy="0.0008" iyz="0" izz="0.0010"/>
-    </inertial>
-  </link>
-  <joint name="sensor_dome_joint" type="fixed">
-    <parent link="base_link"/>
-    <child link="sensor_dome"/>
-    <origin xyz="0.08 0 0.055" rpy="0 0 0"/>
-  </joint>
-  <!-- Dome lens -->
-  <link name="dome_lens">
-    <visual>
-      <geometry><cylinder radius="0.035" length="0.008"/></geometry>
-      <material name="white"/>
-    </visual>
-    <collision>
-      <geometry><cylinder radius="0.001" length="0.001"/></geometry>
-    </collision>
-    <inertial>
-      <mass value="0.01"/>
-      <inertia ixx="0.00001" ixy="0" ixz="0" iyy="0.00001" iyz="0" izz="0.00001"/>
-    </inertial>
-  </link>
-  <joint name="dome_lens_joint" type="fixed">
-    <parent link="sensor_dome"/>
-    <child link="dome_lens"/>
-    <origin xyz="0 0 0.029" rpy="0 0 0"/>
-  </joint>
   <!-- Left wheel -->
   <link name="left_wheel">
@@ -133,24 +49,4 @@
     <origin xyz="0 0.39 -0.06" rpy="0 0 0"/>
     <axis xyz="0 1 0"/>
-  </joint>
-  <!-- Left rim ring -->
-  <link name="left_rim">
-    <visual>
-      <origin xyz="0 0 0" rpy="1.5708 0 0"/>
-      <geometry><cylinder radius="0.085" length="0.080"/></geometry>
-      <material name="orange_rim"/>
-    </visual>
-    <collision>
-      <geometry><box size="0.001 0.001 0.001"/></geometry>
-    </collision>
-    <inertial>
-      <mass value="0.05"/>
-      <inertia ixx="0.0002" ixy="0" ixz="0" iyy="0.0002" iyz="0" izz="0.0003"/>
-    </inertial>
-  </link>
-  <joint name="left_rim_joint" type="fixed">
-    <parent link="left_wheel"/>
-    <child link="left_rim"/>
-    <origin xyz="0 0 0" rpy="0 0 0"/>
   </joint>
   <!-- Right wheel -->
@@ -176,25 +72,5 @@
     <axis xyz="0 1 0"/>
   </joint>
-  <!-- Right rim ring -->
-  <link name="right_rim">
-    <visual>
-      <origin xyz="0 0 0" rpy="1.5708 0 0"/>
-      <geometry><cylinder radius="0.085" length="0.080"/></geometry>
-      <material name="orange_rim"/>
-    </visual>
-    <collision>
-      <geometry><box size="0.001 0.001 0.001"/></geometry>
-    </collision>
-    <inertial>
-      <mass value="0.05"/>
-      <inertia ixx="0.0002" ixy="0" ixz="0" iyy="0.0002" iyz="0" izz="0.0003"/>
-    </inertial>
-  </link>
-  <joint name="right_rim_joint" type="fixed">
-    <parent link="right_wheel"/>
-    <child link="right_rim"/>
-    <origin xyz="0 0 0" rpy="0 0 0"/>
-  </joint>
-  <!-- Skid plate rear -->
+  <!-- Skid plate rear (fore/aft stability support) -->
   <link name="skid_plate">
     <visual>
@@ -215,5 +91,5 @@
     <origin xyz="-0.27 0 -0.1725" rpy="0 0 0"/>
   </joint>
-  <!-- Skid plate front -->
+  <!-- Skid plate front (fore/aft stability support) -->
   <link name="skid_plate_front">
     <visual>
@@ -234,4 +110,5 @@
     <origin xyz="0.27 0 -0.1725" rpy="0 0 0"/>
   </joint>
+  <!-- Friction tuning -->
   <gazebo reference="skid_plate">
     <mu1>0.1</mu1><mu2>0.1</mu2>
@@ -246,4 +123,5 @@
     <mu1>1.0</mu1><mu2>1.0</mu2>
   </gazebo>
+  <!-- Pose publisher -->
   <gazebo>
     <plugin filename="gz-sim-pose-publisher-system"
@@ -254,4 +132,5 @@
     </plugin>
   </gazebo>
+  <!-- Differential drive -->
   <gazebo>
     <plugin filename="gz-sim-diff-drive-system"
@@ -273,27 +152,25 @@
     </plugin>
   </gazebo>
-  <!-- aruco marker -->
-  <!-- Thin plate for the ArUco marker -->
-<link name="aruco_marker_link">
-  <visual>
-    <geometry>
-      <mesh filename="package://cv_robot/materials/meshes/aruco_marker.obj" scale="1 1 1"/>
-    </geometry>
-  </visual>
-  <collision>
-    <geometry>
-      <box size="0.05 0.05 0.001"/>
-    </geometry>
-  </collision>
-  <inertial>
-    <mass value="0.001"/>
-    <inertia ixx="2.1e-7" ixy="0" ixz="0" iyy="2.1e-7" iyz="0" izz="4.1e-7"/>
-  </inertial>
-</link>
-<!-- Attach the marker to your robot frame -->
-<joint name="aruco_marker_joint" type="fixed">
-  <parent link="base_link"/>
-  <child link="aruco_marker_link"/>
-  <origin xyz="0.0 0.0 0.45" rpy="0 0 0"/>
-</joint>
+  <!-- ArUco marker (overhead-camera localization ground truth) -->
+  <link name="aruco_marker_link">
+    <visual>
+      <geometry>
+        <mesh filename="package://cv_robot/materials/meshes/aruco_marker.obj" scale="1 1 1"/>
+      </geometry>
+    </visual>
+    <collision>
+      <geometry>
+        <box size="0.05 0.05 0.001"/>
+      </geometry>
+    </collision>
+    <inertial>
+      <mass value="0.001"/>
+      <inertia ixx="2.1e-7" ixy="0" ixz="0" iyy="2.1e-7" iyz="0" izz="4.1e-7"/>
+    </inertial>
+  </link>
+  <joint name="aruco_marker_joint" type="fixed">
+    <parent link="base_link"/>
+    <child link="aruco_marker_link"/>
+    <origin xyz="0.0 0.0 0.85" rpy="0 0 0"/>
+  </joint>
 </robot>
